Commit message: Add physical proberities of the robot model

File: urdf/RoboMaid.urdf (robot description, URDF)
Before this commit: robot RoboMaid, 5 links, 4 joints
Links:
- link back_roller: mass None -> 0.12; geometry collision sphere radius=0.025; visual sphere radius=0.025
- link base_link: mass None -> 2; geometry collision box size=0.35 0.35 0.005; visual box size=0.35 0.35 0.005
- link front_roller: mass None -> 0.12; geometry collision sphere radius=0.025; visual sphere radius=0.025
- link left_wheel_link: mass None -> 0.2; geometry collision cylinder length=0.035 radius=0.03; visual cylinder length=0.035 radius=0.03
- link right_wheel_link: mass None -> 0.2; geometry collision cylinder length=0.035 radius=0.03; visual cylinder length=0.035 radius=0.03

Commit message: Mount Laser model on Robot  Base

File: urdf/RoboMaid.urdf (robot description, URDF)
Before this commit: robot RoboMaid, 5 links, 4 joints
Links:
- added link base_laser, mass 0.15717; collision mesh filename=package://RoboMaid_sim/meshes/ydlidar.dae; visual mesh filename=package://RoboMaid_sim/meshes/ydlidar.dae
- added link laser_frame, mass 0.25482
Joints:
- added joint base_to_lidar: type continuous, parent base_link, child base_laser, origin xyz=0 0 0, axis 0 0 1
- added joint laser_joint: type fixed, parent base_laser, child laser_frame, origin xyz=0 0 0.03172 rpy=0 0 0, axis 0 0 0

Commit message: Add Gazebo version 1.0

File: urdf/RoboMaid.urdf (robot description, URDF)
Before this commit: robot RoboMaid, 7 links, 6 joints
Joints:
- removed joint base_to_righ_wheel
- added joint base_to_right_wheel: type continuous, parent base_link, child right_wheel_link, origin xyz=0 0.135 -0.02, axis 0 1 0
- joint base_to_left_wheel: origin xyz=0 -0.135 0 -> xyz=0 -0.135 -0.02

Commit message: Add ydlidar plugin

File: urdf/RoboMaid.urdf (robot description, URDF)
Before this commit: robot RoboMaid, 7 links, 6 joints
Joints:
- joint base_to_lidar: type continuous -> fixed
