Commit message: Add slam_karo

File: urdf/no_plugins.urdf.xacro (robot description, xacro)
@@ -222,74 +222,3 @@
 	<origin xyz="0 0 0"/>
   </joint>
-	<!-- adding transmitions for wheels to control their velocity from gazebo -->
-<xacro:macro name="wheel-trans" params="wheel_type">
-    <gazebo reference="${wheel_type}_wheel">
-      <mu1 value="200.0"/>
-      <mu2 value="100.0"/>
-      <kp value="10000000.0" />
-      <kd value="1.0" />
-      <material>Gazebo/Black</material>
-    </gazebo>
-    <!-- This block connects the wheel joint to an actuator (motor), which informs both
-    simulation and visualization of the robot -->
-    <transmission name="${wheel_type}_wheel_trans">
-      <type>transmission_interface/SimpleTransmission</type>
-      <actuator name="${wheel_type}_wheel_motor">
-        <mechanicalReduction>1</mechanicalReduction>
-      </actuator>
-      <joint name="base_to_${wheel_type}_wheel">
-        <hardwareInterface>hardware_interface/VelocityJointInterface</hardwareInterface>
-      </joint>
-    </transmission>
- </xacro:macro>
-<xacro:macro name="wheel-speed-read" params="wheel_type">
-    <transmission name="${wheel_type}_wheel_reading">
-      <type>transmission_interface/SimpleTransmission</type>
-    <joint name="base_to_${wheel_type}_wheel">
-      <hardwareInterface>hardware_interface/PositionJointInterface</hardwareInterface>
-    </joint>
-    </transmission>
- </xacro:macro>
- <xacro:wheel-trans wheel_type="left"/>
- <xacro:wheel-trans wheel_type="right"/>
-<xacro:wheel-speed-read wheel_type="left"/>
-<xacro:wheel-speed-read wheel_type="right"/>
-	<!--Gazebo plugin for lidar -->
-  <gazebo reference="laser_frame">
-    <sensor type="ray" name="ydlidar_X4_sensor">
-      <pose>0 0 0.0 0 0 0</pose>
-      <visualize>false</visualize>
-      <update_rate>40</update_rate>
-      <ray>
-        <scan>
-          <horizontal>
-            <samples>5000</samples>
-            <resolution>1</resolution>
-            <min_angle>-3.14159265359</min_angle>
-            <max_angle>3.14159265359</max_angle>
-          </horizontal>
-        </scan>
-        <range>
-          <min>0.12</min>
-          <max>12.0</max>
-          <resolution>0.5</resolution>
-        </range>
-        <noise>
-          <type>gaussian</type>
-          <mean>0.0</mean>
-          <stddev>0.01</stddev>
-        </noise>
-      </ray>
-      <plugin name="gazebo_ros_ydlidarx4_controller" filename="libgazebo_ros_laser.so">
-        <topicName>/robomaid/laser/scan</topicName>
-        <frameName>laser_frame</frameName>
-      </plugin>
-    </sensor >
-  </gazebo>
-	<!--making ros interact with gazebo-->
-  <gazebo>
-       <plugin name="gazebo_ros_control" filename="libgazebo_ros_control.so">
-          <robotNamespace>/</robotNamespace>
-      </plugin>
-  </gazebo>
 </robot>
