Commit message: Fix sensor issue

File: urdf/RoboMaid.urdf.xacro (robot description, xacro)
@@ -157,5 +157,5 @@
         izz="0.00011103" />
     </inertial>
-    <!--visual>
+    <visual>
       <origin
         xyz="0 0 0"
@@ -170,6 +170,6 @@
           rgba="0.64706 0.61961 0.58824 1" />
       </material>
-    </visual-->
-    <!--collision>
+    </visual>
+    <collision>
       <origin
         xyz="0 0 0"
@@ -179,5 +179,5 @@
           filename="package://ydlidar_ros/meshes/ydlidar.dae" />
       </geometry>
-    </collision-->
+    </collision>
   </link>
   <joint name="base_to_right_wheel" type="continuous">
@@ -256,16 +256,16 @@
 <xacro:wheel-speed-read wheel_type="right"/>
 	<!--Gazebo plugin for lidar -->
-  <gazebo reference="base_laser">
-    <sensor type="gpu_ray" name="ydlidar_X4_sensor">
-      <pose>0 0 0 0 0 0</pose>
-      <visualize>false</visualize>
+  <gazebo reference="laser_frame">
+    <sensor type="ray" name="ydlidar_X4_sensor">
+      <pose>0 0 0.0 0 0 0</pose>
+      <visualize>true</visualize>
       <update_rate>40</update_rate>
       <ray>
         <scan>
           <horizontal>
-            <samples>720</samples>
+            <samples>5000</samples>
             <resolution>1</resolution>
-            <min_angle>-1.570796</min_angle>
-            <max_angle>1.570796</max_angle>
+            <min_angle>-3.14159265359</min_angle>
+            <max_angle>3.14159265359</max_angle>
           </horizontal>
         </scan>
@@ -277,17 +277,13 @@
         <noise>
           <type>gaussian</type>
-          <!-- Noise parameters based on published spec for Hokuyo laser
-               achieving "+-30mm" accuracy at range < 10m.  A mean of 0.0m and
-               stddev of 0.01m will put 99.7% of samples within 0.03m of the true
-               reading. -->
           <mean>0.0</mean>
           <stddev>0.01</stddev>
         </noise>
       </ray>
-      <plugin name="gazebo_ros_ydlidar_controller" filename="libgazebo_ros_gpu_laser.so">
+      <plugin name="gazebo_ros_ydlidarx4_controller" filename="libgazebo_ros_laser.so">
         <topicName>/robomaid/laser/scan</topicName>
-        <frameName>base_laser</frameName>
+        <frameName>laser_frame</frameName>
       </plugin>
-    </sensor>
+    </sensor >
   </gazebo>
 	<!--making ros interact with gazebo-->

Commit message: Remove joint_state_controller

File: urdf/RoboMaid.urdf.xacro (robot description, xacro)
@@ -178,5 +178,5 @@
 	<!-- adding transmitions for wheels to control their velocity from gazebo -->
 <xacro:macro name="wheel-trans" params="wheel_type">
-    <gazebo reference="${wheel_type}_wheel">
+    <gazebo reference="${wheel_type}_wheel_link">
       <mu1 value="200.0"/>
       <mu2 value="100.0"/>
@@ -197,6 +197,8 @@
     </transmission>
  </xacro:macro>
-<xacro:macro name="wheel-speed-read" params="wheel_type">
-    <transmission name="${wheel_type}_wheel_reading">
+ <xacro:wheel-trans wheel_type="left"/>
+ <xacro:wheel-trans wheel_type="right"/>
+<!--<xacro:macro name="wheel_position_state" params="wheel_type">
+    <transmission name="${wheel_type}_wheel_state">
       <type>transmission_interface/SimpleTransmission</type>
     <joint name="base_to_${wheel_type}_wheel">
@@ -204,9 +206,7 @@
     </joint>
     </transmission>
- </xacro:macro>
- <xacro:wheel-trans wheel_type="left"/>
- <xacro:wheel-trans wheel_type="right"/>
-<xacro:wheel-speed-read wheel_type="left"/>
-<xacro:wheel-speed-read wheel_type="right"/>
+ </xacro:macro>-->
+<!--<xacro:wheel_position_state wheel_type="left"/>-->
+<!--<xacro:wheel_position_state wheel_type="right"/>-->
 	<!--Gazebo plugin for lidar -->
   <gazebo reference="laser_frame">

Commit message: putting the wheel in correct position

File: urdf/RoboMaid.urdf.xacro (robot description, xacro)
@@ -141,13 +141,13 @@
     </collision>
   </link>
-  <joint name="base_to_right_wheel" type="continuous">
-	<parent link="base_link"/>
-	<child link="right_wheel_link"/>
+  <joint name="base_to_left_wheel" type="continuous">
+	<parent link="base_link"/>
+	<child link="left_wheel_link"/>
         <axis xyz="0 1 0"/>
 	<origin xyz="0 0.135 -0.02"/>
   </joint>
-  <joint name="base_to_left_wheel" type="continuous">
-	<parent link="base_link"/>
-	<child link="left_wheel_link"/>
+  <joint name="base_to_right_wheel" type="continuous">
+	<parent link="base_link"/>
+	<child link="right_wheel_link"/>
 	<axis xyz="0 1 0"/>
 	<origin xyz="0 -0.135 -0.02"/>
@@ -174,5 +174,5 @@
       link="laser_frame" />
     <axis
-      xyz="0 0 0" />
+      xyz="0  0 1" />
   </joint>
 	<!-- adding transmitions for wheels to control their velocity from gazebo -->

Commit message: Fix position of the front roller so that robot base is straight

File: urdf/RoboMaid.urdf.xacro (robot description, xacro)
@@ -21,5 +21,5 @@
     </collision>
      <inertial>
-	<mass value="2"/>
+	<mass value="2.4"/>
 	<inertia ixx="0.0204" ixy="0.0" ixz="0.0" iyy="0.0408" iyz="0.0" izz="0.0204"/>
      </inertial>
@@ -66,17 +66,18 @@
     <visual>
       <geometry>
-        <sphere  radius="0.025"/>
-      </geometry>
-      <origin  xyz="0 0 -0.025"/>
+        <sphere  radius="0.015"/>
+      </geometry>
+      <origin  xyz="0 0 -0.015"/>
 	<material name="black"/>
     </visual>
      <collision>
 	<geometry>
-        <sphere  radius="0.025"/>
-      </geometry>
-      <origin  xyz="0 0 -0.025"/>
+        <sphere  radius="0.015"/>
+      </geometry>
+      <origin  xyz="0 0 -0.015"/>
+      <mu  value="10"/>
      </collision>
      <inertial>
-	<mass value="0.6"/>
+	<mass value="0.12"/>
 	<inertia ixx="0.00003" ixy="0.0" ixz="0.0" iyy="0.00003" iyz="0.0" izz="0.00003"/>
      </inertial>
@@ -145,5 +146,5 @@
 	<child link="left_wheel_link"/>
         <axis xyz="0 1 0"/>
-	<origin xyz="0 0.135 -0.02"/>
+	<origin xyz="0 0.135 -0.0025"/>
   </joint>
   <joint name="base_to_right_wheel" type="continuous">
@@ -151,10 +152,10 @@
 	<child link="right_wheel_link"/>
 	<axis xyz="0 1 0"/>
-	<origin xyz="0 -0.135 -0.02"/>
+	<origin xyz="0 -0.135 -0.0025"/>
   </joint>
   <joint name="base_to_front_roller" type="fixed">
 	<parent link="base_link"/>
 	<child link="front_roller"/>
-	<origin xyz="-0.14 0 0"/>
+	<origin xyz="0.14 0 -0.0025"/>
   </joint>
   <!--<joint name="base_to_back_roller" type="fixed">
@@ -214,5 +215,5 @@
       <pose>0 0 0.0 0 0 0</pose>
       <visualize>false</visualize>
-      <update_rate>40</update_rate>
+      <update_rate>50</update_rate>
       <ray>
         <scan>

Commit message: Add hector_mapping node

File: urdf/RoboMaid.urdf.xacro (robot description, xacro)
@@ -21,5 +21,5 @@
     </collision>
      <inertial>
-	<mass value="2.4"/>
+	<mass value="2"/>
 	<inertia ixx="0.0204" ixy="0.0" ixz="0.0" iyy="0.0408" iyz="0.0" izz="0.0204"/>
      </inertial>
